File: SUNSOFT-E301.kicad_sch (KiCad schematic)
At the start: 26 parts, among them J1 Famicom Card Edge Connector, U1 HM6264, U2 FME7-5A-5B, U3 27C040, U4 27C020

Commit message: Revision 0.0.4
Parts:
- removed JP1: ~, Jumper:SolderJumper-2_P1.3mm_Open_RoundedPad1.0x1.5mm, symbol Jumper:SolderJumper_2_Open
- added JP1: SolderJumper_2_Bridged, Jumper:SolderJumper-2_P1.3mm_Bridged_RoundedPad1.0x1.5mm, symbol Jumper:SolderJumper_2_Bridged
- added JP5: ~, Jumper:SolderJumper-3_P1.3mm_Open_RoundedPad1.0x1.5mm, symbol Jumper:SolderJumper_3_Open
- added JP6: ~, Jumper:SolderJumper-3_P1.3mm_Bridged12_RoundedPad1.0x1.5mm, symbol Jumper:SolderJumper_3_Bridged12
- added TP1: ~, TestPoint:TestPoint_Pad_D1.0mm, symbol Connector:TestPoint
- U1: footprint Package_DIP:DIP-28_W15.24mm_Socket -> Package_DIP:DIP-28_W15.24mm
- U2: footprint Package_QFP:TQFP-44_10x10mm_P0.8mm -> custom footprints:Sunsoft-5
Connections:
- net AUD_IN: now also JP1.2 (B)
- net AUD_OUT: now also JP1.1 (A)
- net GND: now also JP5.3 (B)
- net PRG_A18: now also JP6.2 (C); no longer JP2.3 (B)
- net VCC: now also JP5.1 (A), JP6.1 (A)
- net at U2.18 (NC): now also JP5.2 (C), TP1.1
- net VCC_BATT: now reaches BT1.1 (+), D2.2 (A)
- new net: JP2.3 (B), JP6.3 (B)
- no-connect marks 4 -> 3
Other:
- note added: "FME-7 / 5A / 5B mapper chip Bridge pads 1 and 2 of all solder jumpers if using a non-FME7 chip (5A, 5B) Otherwise, bridge pads 2 and 3 if applicable If using 512K PRG ROM, cut from VCC and bridge pads 2 and 3"
- note added: "PRG ROM 512K/256K"
- note added: "Pin 18 testing and debugging Keep unconnected when not in use"
- note added: "Sunsoft 5B Audio Circuit If not in use, leave components unoccupied. Otherwise, break EXP. AUD BYPASS bridge before use."
- note added: "Work RAM / Save RAM (8K high speed SRAM) If not in use, don't occupy."
- note removed: "Bridge pads 1 and 2 of all solder jumpers if using a non-FME7 chip (5A, 5B) Otherwise, bridge pads 2 and 3 if applicable"
- note removed: "FME7/5A/5B mapper chip"
- note removed: "PRG ROM 512K"
- note removed: "Sunsoft 5B Audio Circuit"
- note removed: "WRAM (8K high speed SRAM)"
- company: (none) -> Persune
- title: FME7-5A-5B-Devboard -> FME-7 / 5A / 5B DevBoard (SS-E301 / JxROM)
- moved on the sheet: U2
